File: horsie-65.kicad_pcb (KiCad board)
At the start: 2 copper layers, 304.8 x 95.3 mm, 32 parts, among them SW14 BSPC, SW29 \|, SW42 ', SW43 ENTR, SW44 PGUP, SW45 LSHF, SW46 Z, SW47 X, SW48 C, SW49 V, SW50 B, SW51 N, SW52 M, SW53 ,<, SW54 .>, SW55 /?, SW56 RSHF, SW57 UARW, SW58 PGDN, SW59 LCTR, SW60 WNDW, SW61 LALT, SW62 SPCB, SW63 RALT, SW64 FNKY, SW65 LARW, SW66 DARW, SW67 RARW, SW68 SW_Push, U2 ATmega32U4-AU, Y1 Crystal_GND24_Small

Commit message: more pcb
Parts:
- moved SW68 18.1 mm to (194.1, 100.2)
- moved R1 7.94 mm to (128.6, 105.8)
- moved U2 2.51 mm to (176.2, 106.4)
Routing:
- net row0: track 0.00 -> 303.4 mm
- net row1: track 0.00 -> 298.6 mm
- net row4: track 0.00 -> 297.7 mm
- net row2: track 0.00 -> 295.0 mm
- net row3: track 0.00 -> 289.4 mm
- net GND: track 0.00 -> 127.9 mm, vias 0 -> 2
- net col1: track 0.00 -> 95.4 mm
- net col2: track 0.00 -> 91.5 mm
- net col13: track 0.00 -> 87.1 mm
- net +5V: track 0.00 -> 87.0 mm, vias 0 -> 2
- net col11: track 0.00 -> 85.6 mm
- net col0: track 0.00 -> 85.6 mm
- net col12: track 0.00 -> 84.1 mm
- net col14: track 0.00 -> 78.3 mm
- net col8: track 0.00 -> 67.1 mm
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
Commit message: more routing
Parts:
- moved R1 97.9 mm to (226.3, 99.2), turned to 270 degrees
- moved SW68 6.94 mm to (187.7, 97.4), turned to 0 degrees
- moved Y1 1.14 mm to (191.2, 108.6), turned to 90 degrees
Connections:
- U2 pad 1: row0 -> row3
- U2 pad 38: row1 -> row4
- U2 pad 39: row4 -> row0
- U2 pad 40: row3 -> row1
Routing:
- net col0: track 85.6 -> 242.6 mm, vias 0 -> 1
- net col14: track 78.3 -> 225.1 mm, vias 0 -> 1
- net col1: track 95.4 -> 227.3 mm, vias 0 -> 1
- net col13: track 87.1 -> 213.5 mm, vias 0 -> 1
- net col2: track 91.5 -> 198.0 mm, vias 0 -> 1
- net col12: track 84.1 -> 190.0 mm, vias 0 -> 1
- net col3: track 67.0 -> 160.3 mm, vias 0 -> 1
- net col10: track 67.0 -> 144.3 mm, vias 0 -> 1
- net col11: track 85.6 -> 158.7 mm, vias 0 -> 1
- net col4: track 67.0 -> 139.3 mm, vias 0 -> 1
- net col9: track 67.0 -> 125.5 mm, vias 0 -> 1
- net +5V: track 87.0 -> 143.7 mm, vias 2 -> 8
- net col8: track 67.1 -> 117.4 mm, vias 0 -> 1
- net col6: track 67.0 -> 114.2 mm, vias 0 -> 1
- net col5: track 67.0 -> 104.0 mm, vias 0 -> 1
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
Commit message: aesthetics 1
Parts:
- removed R1: 10k, Resistor_SMD:R_0805_2012Metric_Pad1.15x1.40mm_HandSolder
- removed SW68: SW_Push, random-keyboard-parts:SKQG-1155865
- removed U2: ATmega32U4-AU, Package_QFP:TQFP-44_10x10mm_P0.8mm
- removed Y1: Crystal_GND24_Small, Crystal:Crystal_SMD_3225-4Pin_3.2x2.5mm_HandSoldering
- added SW16: TAB, MX_Only:MXOnly-1.5U-NoLED, F.Cu at (38.1, 52.4)
- added SW31: CAPS, MX_Only:MXOnly-1.75U-NoLED, F.Cu at (40.5, 71.4)
Routing:
- net row0: track 303.4 -> 506.0 mm
- net row1: track 298.6 -> 481.1 mm
- net row2: track 295.0 -> 454.8 mm
- net RESET: track 5.61 -> 50.3 mm, vias 0 -> 2
- net MOSI: track 0.00 -> 41.5 mm
- net SCK: track 0.00 -> 39.8 mm
- net +5V: track 143.7 -> 182.6 mm
- net GND: track 161.6 -> 199.8 mm
- net MISO: track 0.00 -> 37.8 mm
- net row3: track 289.4 -> 308.4 mm
- net row4: track 300.8 -> 312.9 mm, vias 0 -> 2
- net D+: track 6.50 -> 7.65 mm
- net D-: track 8.42 -> 9.15 mm
- net col9: track 125.5 -> 126.1 mm
