File: horsie-65.kicad_pcb (KiCad board)
At the start: 2 copper layers, 304.8 x 95.2 mm, 30 parts, among them SW14 BSPC, SW16 TAB, SW29 \|, SW31 CAPS, SW42 ', SW43 ENTR, SW44 PGUP, SW45 LSHF, SW46 Z, SW47 X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

Commit message: feedback fixes
Parts:
- added SW22: Y, MX_Only:MXOnly-1U-NoLED, F.Cu at (191.3, 123.8)
Routing:
- net Net-(D22-Pad2): track 6.82 -> 12.7 mm
- net Net-(D51-Pad2): track 6.82 -> 12.7 mm
- net Net-(D37-Pad2): track 6.82 -> 12.7 mm
- net row4: track 313.7 -> 316.6 mm
- net row3: track 308.5 -> 307.2 mm
- net row2: track 454.9 -> 453.7 mm

Commit message: pre ground fill again
Routing:
- net row0: track 506.0 -> 0.00 mm
- net row1: track 481.3 -> 0.00 mm
- net row2: track 453.7 -> 0.00 mm, vias 2 -> 0
- net row4: track 316.6 -> 0.00 mm, vias 4 -> 0
- net row3: track 307.2 -> 0.00 mm, vias 4 -> 0
- net col0: track 241.6 -> 0.00 mm, vias 1 -> 0
- net col1: track 226.4 -> 0.00 mm, vias 1 -> 0
- net col14: track 225.6 -> 0.00 mm, vias 1 -> 0
- net col13: track 213.5 -> 0.00 mm, vias 1 -> 0
- net GND: track 203.7 -> 0.00 mm, vias 2 -> 0
- net col2: track 197.7 -> 0.00 mm, vias 1 -> 0
- net col12: track 190.0 -> 0.00 mm, vias 1 -> 0
- net +5V: track 188.1 -> 0.00 mm, vias 8 -> 0
- net col3: track 159.0 -> 0.00 mm, vias 1 -> 0
- net col11: track 156.8 -> 0.00 mm, vias 1 -> 0
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Other:
- board outline removed

Commit message: ground fills
Routing:
- added copper zone on B.Cu, net GND
- added copper zone on F.Cu, net GND
Changed lines of the file:
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@@
+    )
+  )
+  (zone (net 1) (net_name GND) (layer B.Cu) (hatch edge 0.508)
+    (connect_pads (clearance 0.1524))
+    (min_thickness 0.254)
+    (fill yes (arc_segments 32) (thermal_gap 0.508) (thermal_bridge_width 0.508))
+    (polygon
+      (pts
+        (xy 57.15 94.45625) (xy 57.15 191.29375) (xy 363.5375 191.29375) (xy 363.5375 94.45625)
+      )
+    )
+  )
+  (zone (net 1) (net_name GND) (layer F.Cu) (hatch edge 0.508)
+    (connect_pads (clearance 0.1524))
+    (min_thickness 0.254)
+    (fill yes (arc_segments 32) (thermal_gap 0.508) (thermal_bridge_width 0.508))
+    (polygon
+      (pts
+        (xy 57.15 94.45625) (xy 57.15 191.29375) (xy 363.5375 191.29375) (xy 363.5375 94.45625)
+      )
     )
   )

Commit message: logos
Parts:
- added G***: LOGO, local:logosmall, F.Cu at (155.6, 178.6)
- added G***: LOGO, local:logo, F.Cu at (223.8, 146.8)
